File: AML_MicIn/AML-07-048.sch (KiCad schematic (older format))
At the start: 66 parts, among them J1 Con, J2 Con, J3 Con, J4 Con, J5 Con, J6 Con, J7 Con, J8 Con, J9 Con, Q1 BC560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

Commit message: fix in MicIn schematic, BJT section of S1000
Connections:
- net GND: now also R2.2, R3.2
- net at C1.1, C3.1, J2.1 (Pin_1)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: no longer R3.2
- net at C1.2, C2.1, J1.1 (Pin_1)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: no longer R2.2
Changed lines of the file:
@@
 	1250 4600 1250 4700
 Wire Wire Line
-	1100 5100 950  5100
-Wire Wire Line
-	950  5100 950  4600
-Wire Wire Line
-	950  3900 950  3400
-Wire Wire Line
-	950  3400 1100 3400
-Connection ~ 950  3900
+	1100 5100 1000 5100
+Wire Wire Line
+	1000 3400 1100 3400
 Wire Wire Line
 	1750 3900 1850 3900
@@
 Wire Wire Line
 	2350 4700 2350 4250
-Connection ~ 950  4600
 Connection ~ 2050 4250
 Connection ~ 2350 4250
@@
 	1    0    0    -1
 $EndComp
+$Comp
+L power:GND #PWR?
+U 1 1 62C27E6F
+P 1000 3400
+F 0 "#PWR?" H 1000 3150 50  0001 C CNN
+F 1 "GND" V 900 3400 50  0000 R CNN
+F 2 "" H 1000 3400 50  0001 C CNN
+F 3 "" H 1000 3400 50  0001 C CNN
+	1    1000 3400
+	0    1    1    0
+$EndComp
+$Comp
+L power:GND #PWR?
+U 1 1 62C3662E
+P 1000 5100
+F 0 "#PWR?" H 1000 4850 50  0001 C CNN
+F 1 "GND" V 900 5100 50  0000 R CNN
+F 2 "" H 1000 5100 50  0001 C CNN
+F 3 "" H 1000 5100 50  0001 C CNN
+	1    1000 5100
+	0    1    1    0
+$EndComp
 $EndSCHEMATC
