File: TAC_RI277/RI277D.sch (KiCad schematic (older format))
At the start: 9 parts, among them J1 Ribbon Cable, J2 Tape Return

Commit message: included RI277 to diagram, fixed missing bridge pin 6-7 on RI277D
Connections:
- net at J1.6 (Pin_6), J2.3 (Pin_3), SK2.RN: now also J1.7 (Pin_7)
- no-connect marks 5 -> 4
Changed lines of the file:
@@
 	3100 2100 3100 3100
 Wire Wire Line
-	3100 3100 4000 3100
+	3100 3100 3950 3100
 Wire Wire Line
 	4000 2000 3500 2000
@@
 NoConn ~ 2600 3800
 NoConn ~ 2600 4000
-NoConn ~ 4000 3200
 NoConn ~ 4000 2800
 Wire Wire Line
@@
 Wire Wire Line
 	3550 2200 3550 2150
+Wire Wire Line
+	4000 3200 3950 3200
+Wire Wire Line
+	3950 3200 3950 3100
+Connection ~ 3950 3100
+Wire Wire Line
+	3950 3100 4000 3100
 $EndSCHEMATC
