File: TAC_GL270D/GL270D.sch (KiCad schematic (older format))
At the start: 15 parts, among them SW1 +48V On, SW2 SW_QPDT_x4, SW3 SW_DPDT_x2, SW4 SW_DPDT_x2

Commit message: fix in MicIn schematic, BJT section of S1000
Parts:
- added C101: 2n2 K100, symbol Device:C
- added C102, C103: 63V 47u, symbol Device:CP
- added C107, C108, C5, C6: 47u, symbol Device:CP
- added D1, D2, D3, D4: 1N4148, symbol Device:D
- added Q103, Q104, Q105, Q106: BC560, Package_TO_SOT_THT:TO-92_Inline, symbol Transistor_BJT:BC560
- added R101: 1k5, symbol Device:R
- added R102, R103: 10k, symbol Device:R
- added R107, R111: 3k3, symbol Device:R
- added R108, R110: 6k8, symbol Device:R
- added R112, R113: 1M, symbol Device:R
- renumbered FB2 to FB1, FB1 to FB2
Connections:
- net labels added: J1, J2
- wire segments 54 -> 126
Other:
- moved on the sheet: J?, R1, R2, SW1

Commit message: fully drawn components of MicIn mod PCB AML-07-048
Parts:
- added C104, C112: 3300u, symbol Device:CP
- added C109, C113, C117, C118: 100n, symbol Device:C
- added C110, C111: 22p, symbol Device:C
- added C114: 47u, symbol Device:CP
- added C115, C116: 100p, symbol Device:C
- added C119: 10p, symbol Device:C
- added C120: 10V 100u, symbol Device:CP
- added D5, D6: 1N4148, symbol Device:D
- added Q101, Q102: BC560, Package_TO_SOT_THT:TO-92_Inline, symbol Transistor_BJT:BC560
- added R104: 82k, symbol Device:R
- added R105, R106, R118, R122: 2k2, symbol Device:R
- added R109, R114: 270R, symbol Device:R
- added R115, R117, R121: 5R6, symbol Device:R
- added R116: 1M, symbol Device:R
- added R119, R120: 3k6, symbol Device:R
- added R123: 100k, symbol Device:R
- added RV15: RLG1k, symbol Device:R_POT
- added U101: TL072, symbol Amplifier_Operational:TL072
- added U102: NE5534, symbol Amplifier_Operational:NE5534
- renumbered C5 to C105, C6 to C106
Connections:
- net labels added: J4,6, J5, J7, J9, V+, V-, VCC, VDD
- wire segments 126 -> 255
- no-connect marks 0 -> 1

Commit message: renamed components of AML pcb section, started drawing Eq section
Parts:
- removed C101: 2n2 K100, symbol Device:C
- removed C102, C103: 63V 47u, symbol Device:CP
- removed C104, C112: 3300u, symbol Device:CP
- removed C105, C106, C107, C108, C114: 47u, symbol Device:CP
- removed C109, C113, C117, C118: 100n, symbol Device:C
- removed C110, C111: 22p, symbol Device:C
- removed C115, C116: 100p, symbol Device:C
- removed C119: 10p, symbol Device:C
- removed C120: 10V 100u, symbol Device:CP
- removed Q101, Q102, Q103, Q104, Q105, Q106: BC560, Package_TO_SOT_THT:TO-92_Inline, symbol Transistor_BJT:BC560
- removed R101: 1k5, symbol Device:R
- removed R102, R103: 10k, symbol Device:R
- removed R104: 82k, symbol Device:R
- removed R105, R106, R118, R122: 2k2, symbol Device:R
- removed R107, R111: 3k3, symbol Device:R
- removed R108, R110: 6k8, symbol Device:R
- removed R109, R114: 270R, symbol Device:R
- removed R112, R113, R116: 1M, symbol Device:R
- removed R115, R117, R121: 5R6, symbol Device:R
- removed R119, R120: 3k6, symbol Device:R
- removed R123: 100k, symbol Device:R
- removed U101: TL072, symbol Amplifier_Operational:TL072
- removed U102: NE5534, symbol Amplifier_Operational:NE5534
- added *R42, R20: 10k, symbol Device:R
- added C11, C12: 3n3, symbol Device:C
- added C13: 10p, symbol Device:C
- added R19: 47k, symbol Device:R
- added R21, R23: 1k5, symbol Device:R
- added RV22: LN22k, symbol Device:R_POT
- added SW5: 6k/12k, symbol Switch:SW_SPST
- added SW7: SW_DPDT_x2, symbol Switch:SW_DPDT_x2
- added U2: TL072, symbol Amplifier_Operational:TL072
Connections:
- net labels added:   2n2    K100, 100k, 100n, 100p, 100u 10V, 10k, 10p, 1M, 1k5, 22p, 270R, 2k2, 3300u, 3k3, 3k6, 47u, 5R6, 63V   47u, 6k8, 82k, BC560, J3, J8, NE5534, TL072
- wire segments 255 -> 279
Other:
- note added: "Microphone Input Modification\nPCB: AML-07-048 (Rev 4)\nby Langley Design"
- note added: "S4\n Phase\n Reverse"
- note removed: "S4\nPhase Reverse"

Commit message: Eq middle section
Parts:
- added *R43, *R44, *R45, *R46, *R47, *R48, *R49: 10k, symbol Device:R
- added C14, C15: 680p, symbol Device:C
- added C16, C19: 10p, symbol Device:C
- added C17, C18: 3n3, symbol Device:C
- added R27, R30: 7k5, symbol Device:R
- added R28, R34: 22k, symbol Device:R
- added R29, R35: 15k, symbol Device:R
- added R36: 4k7, symbol Device:R
- added RV24, RV31: LN22k, symbol Device:R_POT
- added RV25, RV26, RV32, RV33: RLG470k, symbol Device:R_POT
- added unit 1 of U2
- added U3, U4: TL072, symbol Amplifier_Operational:TL072
Connections:
- wire segments 279 -> 362
Other:
- note added: "Gain"
- note added: "HF"
- note added: "MF1"
- note added: "MF2"

Commit message: completed EQ section
Parts:
- added C20, C21: u47, symbol Device:C
- added C22: 100u 25V, symbol Device:CP
- added C23: 10p, symbol Device:C
- added C24: 25V 100u, symbol Device:CP
- added R37: 4k7, symbol Device:R
- added R38, R40: 1k, symbol Device:R
- added R41: 100k, symbol Device:R
- added R50: 47R, symbol Device:R
- added RV39: LN22k, symbol Device:R_POT
- added SW6: 60/120Hz, symbol Switch:SW_SPST
- added unit 1 of U4
- SW5: value 6k/12k -> 6/12kHz
Connections:
- wire segments 362 -> 403
Other:
- note added: "LF"
- note added: "MF1 centre"
- note added: "MF2 centre"
- note added: "Microphone Input Modification\nPCB: AML-07-048 (Rev 4)\nby Langley Design\n\nComponents prefixed # or D are\npart of the AML daughter board."
- note added: "Resistors prefixed * are part of DIL resistor packages."
- note added: "SW7\nEQ in"
- note added: "turnovr freq"
- note removed: "Microphone Input Modification\nPCB: AML-07-048 (Rev 4)\nby Langley Design"

Commit message: included RI277 to diagram, fixed missing bridge pin 6-7 on RI277D
Parts:
- added J1: Ribbon Cable, symbol GL270D-rescue:Conn_01x10-Connector_Generic
- added J2: Tape Return, symbol Connector_Generic:Conn_01x03
- added R2: 1k, symbol Device:R
- added R3: 3k, symbol Device:R
- added SK1: MIC Input, symbol Connector_Generic:Conn_01x03
- added SK2: Line Input, symbol Connector:AudioJack3_Switch
- added SK3: Insert, symbol Connector:AudioJack3_Switch
- added SK4: Direct Out, symbol Connector:AudioJack3_Switch
- J1: renamed from J?; value Conn_01x10 -> Ribbon Cable
Connections:
- net labels added: #J1, #J2, #J3, #J4,6, #J5, #J7, #J8, #J9
- net labels removed: J1, J2, J3, J4,6, J5, J7, J8, J9
- wire segments 403 -> 466
- no-connect marks 1 -> 4
Other:
- note added: "CONNECTOR CARD RI277"
- note added: "Components prefixed # or D are part of the AML daughter board."
- note added: "EQUALISER"
- note added: "MIC AMP"
- note added: "Microphone Input Modification\nPCB: AML-07-048 (Rev 4)\nby Langley Design"
- note added: "PCB: RI277D\nby Riven Hexagon"
- note added: "SCN\nTRR\nTRT\n1 GND\n3 -\n2 +"
- note removed: "Microphone Input Modification\nPCB: AML-07-048 (Rev 4)\nby Langley Design\n\nComponents prefixed # or D are\npart of the AML daughter board."
- moved on the sheet: J1, R1, R2, SW1

Commit message: diagram makeup, updated readme
Parts:
- C20, C21: value u47 -> 100 u47
- C22: value 100u 25V -> 25V 100u
- renumbered R2 to **R2, R3 to **R3
Connections:
- net labels added: 10V      100u
- net labels removed: 100u 10V
Other:
- note added: "Microphone Input Modification\nPCB: AML-07-048 (Rev 4)\nby AML & Langley Design"
- note added: "Resistors prefixed ** are part the RI277 connector card."
- note removed: "Microphone Input Modification\nPCB: AML-07-048 (Rev 4)\nby Langley Design"
Changed lines of the file:
@@
 	13850 2300 13700 2300
 Connection ~ 13850 2500
-$Comp
-L Device:CP #C20
-U 1 1 6344089E
-P 14050 2900
-F 0 "#C20" H 14250 2950 50  0000 C CNN
-F 1 "100u 10V" H 14350 2850 50  0000 C CNN
-F 2 "" H 14088 2750 50  0001 C CNN
-F 3 "~" H 14050 2900 50  0001 C CNN
-	1    14050 2900
-	0    -1   -1   0
-$EndComp
 Wire Wire Line
 	13900 2900 13850 2900
@@
 U 1 1 6346D44C
 P 14250 3100
-F 0 "#R23" V 14150 3000 50  0000 L CNN
+F 0 "#R23" V 14350 3000 50  0000 L CNN
 F 1 "100k" V 14250 3000 50  0000 L CNN
 F 2 "" V 14180 3100 50  0001 C CNN
@@
 $EndComp
 Text Notes 8550 4800 0    50   ~ 0
-Microphone Input Modification\nPCB: AML-07-048 (Rev 4)\nby Langley Design
+Microphone Input Modification\nPCB: AML-07-048 (Rev 4)\nby AML & Langley Design
 $Comp
 L Device:R *R42
@@
 	1    0    0    -1
 $EndComp
-Text Notes 18700 14650 0    50   ~ 0
+Text Notes 18700 14550 0    50   ~ 0
 Resistors prefixed * are part of DIL resistor packages.
 $Comp
@@
 $EndComp
 $Comp
-L Device:C C20
-U 1 1 6314D82F
-P 20550 2150
-F 0 "C20" V 20500 2025 50  0000 C CNN
-F 1 "u47" V 20600 2025 50  0000 C CNN
-F 2 "" H 20588 2000 50  0001 C CNN
-F 3 "~" H 20550 2150 50  0001 C CNN
-	1    20550 2150
-	0    1    1    0
-$EndComp
-$Comp
-L Device:C C21
-U 1 1 631612B7
-P 20950 2150
-F 0 "C21" V 20900 2025 50  0000 C CNN
-F 1 "u47" V 21000 2025 50  0000 C CNN
-F 2 "" H 20988 2000 50  0001 C CNN
-F 3 "~" H 20950 2150 50  0001 C CNN
-	1    20950 2150
-	0    1    1    0
-$EndComp
-$Comp
 L Device:CP C22
 U 1 1 631DF9E4
 P 20550 2750
 F 0 "C22" H 20700 2850 50  0000 R CNN
-F 1 "100u 25V" H 20700 2675 50  0000 R CNN
+F 1 "25V 100u" H 20750 2650 50  0000 R CNN
 F 2 "" H 20588 2600 50  0001 C CNN
 F 3 "~" H 20550 2750 50  0001 C CNN
@@
 	1650 4000 1650 3250
 $Comp
-L Device:R R2
+L Device:R **R2
 U 1 1 62DA61F1
 P 1850 4200
-F 0 "R2" V 1800 4350 50  0000 C CNN
+F 0 "**R2" V 1800 4350 50  0000 C CNN
 F 1 "1k" V 1850 4200 50  0000 C CNN
 F 2 "" V 1780 4200 50  0001 C CNN
@@
 $EndComp
 $Comp
-L Device:R R3
+L Device:R **R3
 U 1 1 62DA6DD8
 P 1850 4300
-F 0 "R3" V 1900 4450 50  0000 C CNN
+F 0 "**R3" V 1900 4100 50  0000 C CNN
 F 1 "3k" V 1850 4300 50  0000 C CNN
 F 2 "" V 1780 4300 50  0001 C CNN
@@
 Text Notes 2950 4550 0    50   ~ 0
 PCB: RI277D\nby Riven Hexagon
+Text Notes 18700 14650 0    50   ~ 0
+Resistors prefixed ** are part the RI277 connector card.
+$Comp
+L Device:C C20
+U 1 1 6314D82F
+P 20550 2150
+F 0 "C20" V 20500 2275 50  0000 C CNN
+F 1 "100  u47" V 20600 2150 50  0000 C CNN
+F 2 "" H 20588 2000 50  0001 C CNN
+F 3 "~" H 20550 2150 50  0001 C CNN
+	1    20550 2150
+	0    1    1    0
+$EndComp
+$Comp
+L Device:C C21
+U 1 1 631612B7
+P 20950 2150
+F 0 "C21" V 20900 2275 50  0000 C CNN
+F 1 "100  u47" V 21000 2150 50  0000 C CNN
+F 2 "" H 20988 2000 50  0001 C CNN
+F 3 "~" H 20950 2150 50  0001 C CNN
+	1    20950 2150
+	0    1    1    0
+$EndComp
+$Comp
+L Device:CP #C20
+U 1 1 6344089E
+P 14050 2900
+F 0 "#C20" H 14250 2850 50  0000 C CNN
+F 1 "10V      100u" H 14075 2950 50  0000 C CNN
+F 2 "" H 14088 2750 50  0001 C CNN
+F 3 "~" H 14050 2900 50  0001 C CNN
+	1    14050 2900
+	0    -1   -1   0
+$EndComp
 $EndSCHEMATC

Commit message: completed overload and part of PFL switching section
Parts:
- added *R100, *R52 (x2), *R53, *R54, *R99, R70, R72, R74: 10k, symbol Device:R
- added C25, C26, C27, C29: 25V 100u, symbol Device:CP
- added C28: 10p, symbol Device:C
- added C30: 63V 2u2, symbol Device:CP
- added CR5: RD, symbol Device:LED
- added CR6: YL, symbol Device:LED
- added CR7: 1N4148, symbol Device:D
- added J3: Taper Fader, symbol Connector_Generic:Conn_01x04
- added Q1, Q2: 2N3904, digikey-footprints:TO-92-3, symbol dk_Transistors-Bipolar-BJT-Single:2N3904
- added Q3: 2N3906, digikey-footprints:TO-92-3, symbol dk_Transistors-Bipolar-BJT-Single:2N3906
- added R59: 22k, symbol Device:R
- added R64: 47R, symbol Device:R
- added R65, R71, R73: 1k, symbol Device:R
- added R75: 470R, symbol Device:R
- added R76: 3k, symbol Device:R
- added SW16, SW17: SW_DPDT_x2, symbol Switch:SW_DPDT_x2
- added U5: TL072, symbol Amplifier_Operational:TL072
- renumbered J1 to **J1, J2 to **J2, J1 to J2
Connections:
- net labels added: 1, 2, to_S8_S9
- wire segments 466 -> 567
- no-connect marks 4 -> 6
Other:
- note added: "Components prefixed ** are part the RI277 connector card."
- note added: "OVERLOAD"
- note added: "PFL/AFL\nCONTROL"
- note added: "PFL/AFL\nSIGNAL"
- note added: "SW16\nMUTE"
- note added: "SW17\n PFL"
- note removed: "Resistors prefixed ** are part the RI277 connector card."
