File: TAC_GL270D/GL270D.sch (KiCad schematic (older format))
At the start: 114 parts, among them J2 Ribbon Cable, J3 Taper Fader, Q1 2N3904, Q2 2N3904, Q3 2N3906, SW1 +48V On, SW16 SW_DPDT_x2, SW17 SW_DPDT_x2, SW2 SW_QPDT_x4, SW3 SW_DPDT_x2, SW4 SW_DPDT_x2, SW5 6/12kHz, SW6 60/120Hz, SW7 SW_DPDT_x2, U2 TL072, U3 TL072, U4 TL072, U5 TL072

Commit message: completed PAN section and S1100 aux send option
Parts:
- added *R105, *R106, *R107, *R108, *R55, *R56, *R57, *R58, *R97, *R98: 10k, symbol Device:R
- added A5, A6, A7, A8, B5, B6, B7, B8: Conn_01x01_Male, symbol Connector:Conn_01x01_Male
- added R101, R102, R103, R104, R66, R67, R68, R69: LG10k, symbol Device:R_POT
- added R60, R61: 2k2, symbol Device:R
- added R62, R63: LN10k, symbol Device:R_POT
- added SW14, SW15: SW_DPDT_x2, symbol Switch:SW_DPDT_x2
- added SW8, SW9: POST/PRE, symbol Switch:SW_SPDT
- J3: value Taper Fader -> (10k)
- renumbered RV15 to R15, RV22 to R22, RV24 to R24, RV25 to R25, RV26 to R26, RV31 to R31, RV32 to R32, RV33 to R33, RV39 to R39
Connections:
- net labels added: 21, 22, 23, 24, 3, 4, 5, 6, 7, 8
- net labels removed: to_S8_S9
- wire segments 567 -> 678
- no-connect marks 6 -> 8
Other:
- note added: "8 AUX SEND OPTION"
- note added: "A5-A8 wired pins"
- note added: "AUDIO\nTAPER\nFADER"
- note added: "AUX 1"
- note added: "AUX 2"
- note added: "AUX 3"
- note added: "AUX 4"
- note added: "L"
- note added: "OVERLOAD DETECT"
- note added: "PAN"
- note added: "R"
- note added: "S1100"
- note removed: "OVERLOAD"

Commit message: completed switching section. Have to revise pin and resistor accociation
Parts:
- added *R77, *R78, *R79, *R80, *R81, *R82, *R83, *R84, *R85, *R86, *R87, *R88, *R89, *R90, *R91, *R92, *R? (x4): 10k, symbol Device:R
- added SW10, SW11, SW12, SW13: SW_QPDT_x4, symbol TAC:SW_QPDT_x4
- CR6: value YL -> RD
- renumbered *R52 to *R51
Connections:
- net labels added: 10, 13, 14, 15, 16, 17, 18, 19, 20, 9
- wire segments 678 -> 761
- no-connect marks 8 -> 28
Other:
- note added: "*DIL"
- note added: "1"
- note added: "10"
- note added: "2"
- note added: "3"
- note added: "4"
- note added: "5"
- note added: "6"
- note added: "7"
- note added: "8"
- note added: "9"
- note added: "SW10\n 1+2\n(9+10)"
- note added: "SW11\n 3+4\n(11+12)"
- note added: "SW12\n 5+6\n(13+14)"
- note added: "SW13\n 7+8\n(15+16)"
- note added: "SW14\n 1-8\n(9-16)"
- note added: "SW15\nSTEREO"
- moved on the sheet: **J1, J2, R1, R2, SW1

Commit message: revised pin assignment DIN 8-12. Need to verify DIN 13-20
Parts:
- renumbered *R97 to *R95, *R98 to *R96
Changed lines of the file:
@@
 Connection ~ 10950 10700
 $Comp
-L Device:R *R97
+L Device:R *R95
 U 1 1 66E2DF21
 P 11650 9500
-F 0 "*R97" V 11550 9400 50  0000 L CNN
+F 0 "*R95" V 11550 9400 50  0000 L CNN
 F 1 "10k" V 11650 9425 50  0000 L CNN
 F 2 "" V 11580 9500 50  0001 C CNN
@@
 	11900 10250 11900 10350
 $Comp
-L Device:R *R98
+L Device:R *R96
 U 1 1 66E2DAD1
 P 11900 10500
-F 0 "*R98" V 11800 10400 50  0000 L CNN
+F 0 "*R96" V 11800 10400 50  0000 L CNN
 F 1 "10k" V 11900 10425 50  0000 L CNN
 F 2 "" V 11830 10500 50  0001 C CNN
