File: TAC_GL270D/GL270-LineIn.sch (KiCad schematic (older format))
At the start: 172 parts, among them J2 Ribbon Cable, J3 (10k), Q1 2N3904, Q2 2N3904, Q3 2N3906, SW1 +48V On, SW10 SW_QPDT_x4, SW11 SW_QPDT_x4, SW12 SW_QPDT_x4, SW13 SW_QPDT_x4, SW14 SW_DPDT_x2, SW15 SW_DPDT_x2, SW16 SW_DPDT_x2, SW17 SW_DPDT_x2, SW2 SW_QPDT_x4, SW3 SW_DPDT_x2, SW4 SW_DPDT_x2, SW5 6/12kHz, SW6 60/120Hz, SW7 SW_DPDT_x2, SW8 POST/PRE, SW9 POST/PRE, U2 TL072, U3 TL072, U4 TL072, U5 TL072

Commit message: completed MicIn diagram
Parts:
- added **J0: to GND wire, symbol Connector:Conn_01x01_Female
- added C31, C32: 25V 220u, symbol Device:CP
- added CR8, CR9: 1N4001, symbol Device:D
- added J?: Conn_01x04_Female, symbol Connector:Conn_01x04_Female
- added R101: 10k, symbol Device:R_POT
- U2, U3, U4, U5: value TL072 -> LM4562
- gave numbers to parts that had none: 4
Connections:
- net labels added: 12, 25, 26, 27, 28, 29, LM4562
- net labels removed: x
- wire segments 762 -> 804
- no-connect marks 28 -> 29
Other:
- note added: "+17.5 V"
- note added: "+V"
- note added: "-17.5 V"
- note added: "-V"
- note added: "0 V"
- note added: "11"
- note added: "12"
- note added: "POWER\nDISTRIBUTION"
- note added: "U2C-U5C"
- note added: "soldered to\nGND wire"
- note added: "wired pins"
- note removed: "16"
- note removed: "A5-A8 wired pins"

Commit message: completed MicIn and LineIn circuit diagrams and fixed errors.
Parts:
- removed D1, D2, D3, D4, D5, D6: 1N4148, symbol Device:D
- removed R1, R2: 6k8, symbol GL270D-rescue:R-Device
- removed R8: 820R, symbol Device:R
- added C10, C12: 63V 22u, symbol Device:CP
- added C6: 10V 220u, symbol Device:CP
- added U25: LM4562, symbol Amplifier_Operational:TL072
- R15: value RLG1k -> LN22k
- R20: value 10k -> 47k
- R3, R4: value 470R -> 4k7
- R36, R37: value 4k7 -> 47k
- R5: value 100R -> 3k9
- R6, R7: value 10k -> 0R
- renumbered R101 to R109
Connections:
- net labels added: #J10, #J4, #J6, 10V      220u, 1k8, 220p, 63V   22u
- net labels removed:   2n2    K100, #J4,6, 100p, 10V      100u, 10p, 1M, 1k5, 270R, 2k2, 3300u, 3k3, 3k6, 47u, 63V   47u, 6k8, 82k, BC560, LM4562, NE5534, V+, V-
- wire segments 804 -> 673
Other:
- note added: "Components prefixed # are part of the AML daughter board."
- note added: "LINE PREAMP"
- note added: "Line Input Mod"
- note added: "Line Input Modification\nPCB: AML-07-046 (Rev 3)\nby AML & Langley Design"
- note added: "SW12\n 5+6\n"
- note added: "SW13\n 7+8\n"
- note added: "SW2\n-10dB PAD"
- note removed: "Components prefixed # or D are part of the AML daughter board."
- note removed: "MIC AMP"
- note removed: "Microphone Input Modification\nPCB: AML-07-048 (Rev 4)\nby AML & Langley Design"
- note removed: "SW12\n 5+6\n(13+14)"
- note removed: "SW13\n 7+8\n(15+16)"
- note removed: "SW2\n-20dB PAD"
