File: TAC_GL270D/GL270-MicIn.sch (KiCad schematic (older format))
At the start: 172 parts, among them J2 Ribbon Cable, J3 (10k), Q1 2N3904, Q2 2N3904, Q3 2N3906, SW1 +48V On, SW10 SW_QPDT_x4, SW11 SW_QPDT_x4, SW12 SW_QPDT_x4, SW13 SW_QPDT_x4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

Commit message: completed MicIn diagram
Parts:
- added **J0: to GND wire, symbol Connector:Conn_01x01_Female
- added C31, C32: 25V 220u, symbol Device:CP
- added CR8, CR9: 1N4001, symbol Device:D
- added J?: Conn_01x04_Female, symbol Connector:Conn_01x04_Female
- added R101: 10k, symbol Device:R_POT
- U2, U3, U4, U5: value TL072 -> LM4562
- gave numbers to parts that had none: 4
Connections:
- net labels added: 11, 12, 25, 26, 27, 28, 29, LM4562
- wire segments 761 -> 804
- no-connect marks 28 -> 29
Other:
- note added: "+17.5 V"
- note added: "+V"
- note added: "-17.5 V"
- note added: "-V"
- note added: "0 V"
- note added: "11"
- note added: "12"
- note added: "POWER\nDISTRIBUTION"
- note added: "U2C-U5C"
- note added: "soldered to\nGND wire"
- note added: "wired pins"
- note removed: "A5-A8 wired pins"

Commit message: completed MicIn and LineIn circuit diagrams and fixed errors.
Parts:
- R20: value 10k -> 47k
- R36, R37: value 4k7 -> 47k
- renumbered R101 to R109
Connections:
- net labels added: #J4, #J6
- net labels removed: #J4,6
- wire segments 804 -> 807
Other:
- note added: "MIC PREAMP"
- note added: "Mic Input Mod"
- note added: "SW12\n 5+6\n"
- note added: "SW13\n 7+8\n"
- note removed: "MIC AMP"
- note removed: "SW12\n 5+6\n(13+14)"
- note removed: "SW13\n 7+8\n(15+16)"
