File: AML_LineIn/AML-07-046.sch (KiCad schematic (older format))
At the start: 36 parts, among them J1 con, J10 Conn_01x01, J2 Con, J3 Con, J4 Con, J5 Con, J6 Con, J7 V+, J8 V-, J9 Conn_01x01, U1 TL072

Commit message: renamed LineIn jumpers, image cleanup
Parts:
- renumbered J3 to J10, J4 to J3, J10 to J4, J8 to J5, J9 to J6, J5 to J8, J6 to J9
Changed lines of the file:
@@
 $EndComp
 $Comp
-L Connector_Generic:Conn_01x01 J8
+L Connector_Generic:Conn_01x01 J5
 U 1 1 60F624B8
 P 1450 2150
-F 0 "J8" H 1530 2192 50  0000 L CNN
+F 0 "J5" H 1530 2192 50  0000 L CNN
 F 1 "V-" H 1400 2050 50  0000 L CNN
 F 2 "" H 1450 2150 50  0001 C CNN
@@
 	3250 2650 3250 2550
 $Comp
-L Connector_Generic:Conn_01x01 J10
+L Connector_Generic:Conn_01x01 J4
 U 1 1 60FB9483
 P 2700 3100
-F 0 "J10" H 2780 3142 50  0000 L CNN
+F 0 "J4" H 2780 3142 50  0000 L CNN
 F 1 "Conn_01x01" H 2300 3000 50  0000 L CNN
 F 2 "" H 2700 3100 50  0001 C CNN
@@
 $EndComp
 $Comp
-L Connector_Generic:Conn_01x01 J9
+L Connector_Generic:Conn_01x01 J6
 U 1 1 60FB9AC3
 P 3000 3100
-F 0 "J9" H 3080 3142 50  0000 L CNN
+F 0 "J6" H 3080 3142 50  0000 L CNN
 F 1 "Conn_01x01" H 2600 3000 50  0000 L CNN
 F 2 "" H 3000 3100 50  0001 C CNN
@@
 	3000 3400 3000 3300
 $Comp
-L Connector_Generic:Conn_01x01 J6
+L Connector_Generic:Conn_01x01 J9
 U 1 1 610331DC
 P 6100 4500
-F 0 "J6" H 6180 4542 50  0000 L CNN
+F 0 "J9" H 6180 4542 50  0000 L CNN
 F 1 "Con" H 6050 4650 50  0000 L CNN
 F 2 "" H 6100 4500 50  0001 C CNN
@@
 	5100 4500 4850 4500
 $Comp
-L Connector_Generic:Conn_01x01 J4
+L Connector_Generic:Conn_01x01 J3
 U 1 1 6106068D
 P 5100 3800
-F 0 "J4" H 5180 3842 50  0000 L CNN
+F 0 "J3" H 5180 3842 50  0000 L CNN
 F 1 "Con" H 5000 3700 50  0000 L CNN
 F 2 "" H 5100 3800 50  0001 C CNN
@@
 $EndComp
 $Comp
-L Connector_Generic:Conn_01x01 J5
+L Connector_Generic:Conn_01x01 J8
 U 1 1 610C203E
 P 3800 4400
-F 0 "J5" H 3880 4442 50  0000 L CNN
+F 0 "J8" H 3880 4442 50  0000 L CNN
 F 1 "Con" H 3700 4550 50  0000 L CNN
 F 2 "" H 3800 4400 50  0001 C CNN
@@
 	4300 4500 4300 4400
 $Comp
-L Connector_Generic:Conn_01x01 J3
+L Connector_Generic:Conn_01x01 J10
 U 1 1 612623AD
 P 4300 3800
-F 0 "J3" H 4380 3842 50  0000 L CNN
+F 0 "J10" H 4380 3842 50  0000 L CNN
 F 1 "Con" H 4200 3950 50  0000 L CNN
 F 2 "" H 4300 3800 50  0001 C CNN

Commit message: completed MicIn and LineIn circuit diagrams and fixed errors.
Connections:
- net GND: now also C10.2; no longer C10.1
- net at J7.1 (Pin_1), R11.2: now also C10.1; no longer C10.2
Changed lines of the file:
@@
 F 3 "~" H 3950 2400 50  0001 C CNN
 	1    3950 2400
-	-1   0    0    1
+	-1   0    0    -1
 $EndComp
 $Comp
