File: DOA_SK25RHX/SK25.sch (KiCad schematic (older format))
At the start: 38 parts, among them Q1 BC560C, Q10 BD140, Q2 KSA992, Q3 KSA992, Q4 BC550C, Q5 BC550C, Q6 BC550C, Q7 BC556C, Q8 BC546C, Q9 BD139

Commit message: completed foot print assignment for DOA SK25
Parts:
- C1, C2: footprint (none) -> Capacitor_THT:C_Disc_D5.0mm_W2.5mm_P2.50mm
- D1, D2, D7, D8, D9: footprint (none) -> Diode_THT:D_DO-35_SOD27_P2.54mm_Vertical_KathodeUp
- D3: footprint (none) -> LED_THT:LED_D3.0mm
- D4: footprint (none) -> Diode_THT:D_DO-35_SOD27_P2.54mm_Vertical_AnodeUp
- D5, D6: footprint (none) -> Diode_THT:D_DO-35_SOD27_P10.16mm_Horizontal
- L1: footprint (none) -> Inductor_THT:L_Axial_L6.6mm_D2.7mm_P2.54mm_Vertical_Vishay_IM-2
- Q1, Q2, Q3, Q4, Q5, Q6, Q7, Q8: footprint (none) -> Package_TO_SOT_THT:TO-92
- Q10, Q9: footprint (none) -> Package_TO_SOT_THT:TO-220-3_Vertical
- R1, R10, R11, R12, R13, R2, R3, R4, R5, R6, R7, R8, R9: footprint (none) -> Resistor_THT:R_Axial_DIN0207_L6.3mm_D2.5mm_P2.54mm_Vertical
- RV1, RV4, RV5: footprint (none) -> Potentiometer_THT:Potentiometer_Bourns_3266Z_Horizontal
Changed lines of the file:
@@
 encoding utf-8
 Sheet 1 1
-Title ""
-Date ""
-Rev ""
-Comp ""
-Comment1 ""
-Comment2 ""
+Title "SK25 Discrete Op-Amp"
+Date "2022-07-31"
+Rev "1.2"
+Comp "Sound Skulptor, Riven Hexagon"
+Comment1 "PCB Layout by Riven Hexagon, 2022"
+Comment2 "Circuit by Sound Skulptor, 2007"
 Comment3 ""
 Comment4 ""
@@
 F 0 "D1" V 2150 3050 50  0000 L CNN
 F 1 "1N914" V 2250 2900 50  0000 L CNN
-F 2 "" H 2200 3250 50  0001 C CNN
+F 2 "Diode_THT:D_DO-35_SOD27_P2.54mm_Vertical_KathodeUp" H 2200 3250 50  0001 C CNN
 F 3 "~" H 2200 3250 50  0001 C CNN
 	1    2200 3250
@@
 F 0 "D2" V 2396 3170 50  0000 R CNN
 F 1 "1N914" V 2305 3170 50  0000 R CNN
-F 2 "" H 2350 3250 50  0001 C CNN
+F 2 "Diode_THT:D_DO-35_SOD27_P2.54mm_Vertical_KathodeUp" H 2350 3250 50  0001 C CNN
 F 3 "~" H 2350 3250 50  0001 C CNN
 	1    2350 3250
@@
 F 0 "Q2" H 3100 3400 50  0000 L CNN
 F 1 "KSA992" H 3100 3500 50  0000 L CNN
-F 2 "" H 3100 3600 50  0001 C CNN
+F 2 "Package_TO_SOT_THT:TO-92" H 3100 3600 50  0001 C CNN
 F 3 "~" H 2900 3500 50  0001 C CNN
 	1    2900 3500
@@
 F 0 "Q3" H 4300 3400 50  0000 L CNN
 F 1 "KSA992" H 4300 3500 50  0000 L CNN
-F 2 "" H 4300 3600 50  0001 C CNN
+F 2 "Package_TO_SOT_THT:TO-92" H 4300 3600 50  0001 C CNN
 F 3 "~" H 4100 3500 50  0001 C CNN
 	1    4100 3500
@@
 F 0 "L1" V 3600 3200 50  0000 C CNN
 F 1 "22µH" V 3450 3200 50  0000 C CNN
-F 2 "" H 3500 3200 50  0001 C CNN
+F 2 "Inductor_THT:L_Axial_L6.6mm_D2.7mm_P2.54mm_Vertical_Vishay_IM-2" H 3500 3200 50  0001 C CNN
 F 3 "~" H 3500 3200 50  0001 C CNN
 	1    3500 3200
@@
 F 0 "R2" H 2850 2800 50  0000 L CNN
 F 1 "100R" H 2750 2700 50  0000 L CNN
-F 2 "" V 2930 2750 50  0001 C CNN
+F 2 "Resistor_THT:R_Axial_DIN0207_L6.3mm_D2.5mm_P2.54mm_Vertical" V 2930 2750 50  0001 C CNN
 F 3 "~" H 3000 2750 50  0001 C CNN
 	1    3000 2750
@@
 F 0 "Q1" H 3791 2154 50  0000 L CNN
 F 1 "BC560C" H 3791 2245 50  0000 L CNN
-F 2 "" H 3800 2300 50  0001 C CNN
+F 2 "Package_TO_SOT_THT:TO-92" H 3800 2300 50  0001 C CNN
 F 3 "~" H 3600 2200 50  0001 C CNN
 	1    3600 2200
@@
 F 0 "R1" V 3793 1500 50  0000 C CNN
 F 1 "470R" V 3884 1500 50  0000 C CNN
-F 2 "" V 3930 1500 50  0001 C CNN
+F 2 "Resistor_THT:R_Axial_DIN0207_L6.3mm_D2.5mm_P2.54mm_Vertical" V 3930 1500 50  0001 C CNN
 F 3 "~" H 4000 1500 50  0001 C CNN
 	1    4000 1500
@@
 F 0 "R6" H 4570 2796 50  0000 L CNN
 F 1 "22k" H 4570 2705 50  0000 L CNN
-F 2 "" V 4430 2750 50  0001 C CNN
+F 2 "Resistor_THT:R_Axial_DIN0207_L6.3mm_D2.5mm_P2.54mm_Vertical" V 4430 2750 50  0001 C CNN
 F 3 "~" H 4500 2750 50  0001 C CNN
 	1    4500 2750
@@
 F 0 "Q5" H 4091 4446 50  0000 L CNN
 F 1 "BC550C" H 4091 4355 50  0000 L CNN
-F 2 "" H 4100 4500 50  0001 C CNN
+F 2 "Package_TO_SOT_THT:TO-92" H 4100 4500 50  0001 C CNN
 F 3 "~" H 3900 4400 50  0001 C CNN
 	1    3900 4400
@@
 F 0 "Q4" H 3291 4446 50  0000 L CNN
 F 1 "BC550C" H 3291 4355 50  0000 L CNN
-F 2 "" H 3300 4500 50  0001 C CNN
+F 2 "Package_TO_SOT_THT:TO-92" H 3300 4500 50  0001 C CNN
 F 3 "~" H 3100 4400 50  0001 C CNN
 	1    3100 4400
@@
 F 0 "R3" H 4070 2796 50  0000 L CNN
 F 1 "100R" H 4070 2705 50  0000 L CNN
-F 2 "" V 3930 2750 50  0001 C CNN
+F 2 "Resistor_THT:R_Axial_DIN0207_L6.3mm_D2.5mm_P2.54mm_Vertical" V 3930 2750 50  0001 C CNN
 F 3 "~" H 4000 2750 50  0001 C CNN
 	1    4000 2750
@@
 F 0 "D3" V 4539 1632 50  0000 R CNN
 F 1 "red" V 4448 1632 50  0000 R CNN
-F 2 "" H 4500 1750 50  0001 C CNN
+F 2 "LED_THT:LED_D3.0mm" H 4500 1750 50  0001 C CNN
 F 3 "~" H 4500 1750 50  0001 C CNN
 	1    4500 1750
@@
 F 0 "R7" V 5650 4000 50  0000 C CNN
 F 1 "39R" V 5850 4000 50  0000 C CNN
-F 2 "" V 5680 4000 50  0001 C CNN
+F 2 "Resistor_THT:R_Axial_DIN0207_L6.3mm_D2.5mm_P2.54mm_Vertical" V 5680 4000 50  0001 C CNN
 F 3 "~" H 5750 4000 50  0001 C CNN
 	1    5750 4000
@@
 F 0 "C1" V 6100 4000 50  0000 C CNN
 F 1 "100pF" V 6400 4000 50  0000 C CNN
-F 2 "" H 6288 3850 50  0001 C CNN
+F 2 "Capacitor_THT:C_Disc_D5.0mm_W2.5mm_P2.50mm" H 6288 3850 50  0001 C CNN
 F 3 "~" H 6250 4000 50  0001 C CNN
 	1    6250 4000
@@
 F 0 "Q7" H 6591 2154 50  0000 L CNN
 F 1 "BC556C" H 6591 2245 50  0000 L CNN
-F 2 "" H 6600 2300 50  0001 C CNN
+F 2 "Package_TO_SOT_THT:TO-92" H 6600 2300 50  0001 C CNN
 F 3 "~" H 6400 2200 50  0001 C CNN
 	1    6400 2200
@@
 F 0 "R9" H 6570 1796 50  0000 L CNN
 F 1 "220R" H 6570 1705 50  0000 L CNN
-F 2 "" V 6430 1750 50  0001 C CNN
+F 2 "Resistor_THT:R_Axial_DIN0207_L6.3mm_D2.5mm_P2.54mm_Vertical" V 6430 1750 50  0001 C CNN
 F 3 "~" H 6500 1750 50  0001 C CNN
 	1    6500 1750
@@
 F 0 "D6" V 6546 3670 50  0000 R CNN
 F 1 "1N914" V 6455 3670 50  0000 R CNN
-F 2 "" H 6500 3750 50  0001 C CNN
+F 2 "Diode_THT:D_DO-35_SOD27_P10.16mm_Horizontal" H 6500 3750 50  0001 C CNN
 F 3 "~" H 6500 3750 50  0001 C CNN
 	1    6500 3750
@@
 F 0 "D5" V 6546 2670 50  0000 R CNN
 F 1 "1N914" V 6455 2670 50  0000 R CNN
-F 2 "" H 6500 2750 50  0001 C CNN
+F 2 "Diode_THT:D_DO-35_SOD27_P10.16mm_Horizontal" H 6500 2750 50  0001 C CNN
 F 3 "~" H 6500 2750 50  0001 C CNN
 	1    6500 2750
@@
 F 0 "R10" H 6570 3296 50  0000 L CNN
 F 1 "22R" H 6570 3205 50  0000 L CNN
-F 2 "" V 6430 3250 50  0001 C CNN
+F 2 "Resistor_THT:R_Axial_DIN0207_L6.3mm_D2.5mm_P2.54mm_Vertical" V 6430 3250 50  0001 C CNN
 F 3 "~" H 6500 3250 50  0001 C CNN
 	1    6500 3250
@@
 F 0 "D8" V 6950 3600 50  0000 L CNN
 F 1 "1N914" V 7050 3600 50  0000 L CNN
-F 2 "" H 7000 3500 50  0001 C CNN
+F 2 "Diode_THT:D_DO-35_SOD27_P2.54mm_Vertical_KathodeUp" H 7000 3500 50  0001 C CNN
 F 3 "~" H 7000 3500 50  0001 C CNN
 	1    7000 3500
@@
 F 0 "Q10" H 7650 3950 50  0000 L CNN
 F 1 "BD140" H 7650 4050 50  0000 L CNN
-F 2 "" H 7600 4100 50  0001 C CNN
+F 2 "Package_TO_SOT_THT:TO-220-3_Vertical" H 7600 4100 50  0001 C CNN
 F 3 "~" H 7400 4000 50  0001 C CNN
 	1    7400 4000
@@
 F 0 "Q9" H 7650 2550 50  0000 L CNN
 F 1 "BD139" H 7650 2450 50  0000 L CNN
-F 2 "" H 7600 2600 50  0001 C CNN
+F 2 "Package_TO_SOT_THT:TO-220-3_Vertical" H 7600 2600 50  0001 C CNN
 F 3 "~" H 7400 2500 50  0001 C CNN
 	1    7400 2500
@@
 F 0 "R12" H 7570 3046 50  0000 L CNN
 F 1 "5R6" H 7570 2955 50  0000 L CNN
-F 2 "" V 7430 3000 50  0001 C CNN
+F 2 "Resistor_THT:R_Axial_DIN0207_L6.3mm_D2.5mm_P2.54mm_Vertical" V 7430 3000 50  0001 C CNN
 F 3 "~" H 7500 3000 50  0001 C CNN
 	1    7500 3000
@@
 F 0 "R13" H 7570 3546 50  0000 L CNN
 F 1 "5R6" H 7570 3455 50  0000 L CNN
-F 2 "" V 7430 3500 50  0001 C CNN
+F 2 "Resistor_THT:R_Axial_DIN0207_L6.3mm_D2.5mm_P2.54mm_Vertical" V 7430 3500 50  0001 C CNN
 F 3 "~" H 7500 3500 50  0001 C CNN
 	1    7500 3500
@@
 F 0 "RV1" H 3430 1704 50  0000 R CNN
 F 1 "2k" H 3430 1795 50  0000 R CNN
-F 2 "" H 3500 1750 50  0001 C CNN
+F 2 "Potentiometer_THT:Potentiometer_Bourns_3266Z_Horizontal" H 3500 1750 50  0001 C CNN
 F 3 "~" H 3500 1750 50  0001 C CNN
 	1    3500 1750
@@
 F 0 "RV4" H 2930 5296 50  0000 R CNN
 F 1 "2k" H 2930 5205 50  0000 R CNN
-F 2 "" H 3000 5250 50  0001 C CNN
+F 2 "Potentiometer_THT:Potentiometer_Bourns_3266Z_Horizontal" H 3000 5250 50  0001 C CNN
 F 3 "~" H 3000 5250 50  0001 C CNN
 	1    3000 5250
@@
 F 0 "D4" V 4450 5350 50  0000 L CNN
 F 1 "Z5V1" V 4550 5350 50  0000 L CNN
-F 2 "" H 4500 5250 50  0001 C CNN
+F 2 "Diode_THT:D_DO-35_SOD27_P2.54mm_Vertical_AnodeUp" H 4500 5250 50  0001 C CNN
 F 3 "~" H 4500 5250 50  0001 C CNN
 	1    4500 5250
@@
 F 0 "Q6" H 4850 4500 50  0000 L CNN
 F 1 "BC550C" H 4850 4600 50  0000 L CNN
-F 2 "" H 5300 4500 50  0001 C CNN
+F 2 "Package_TO_SOT_THT:TO-92" H 5300 4500 50  0001 C CNN
 F 3 "~" H 5100 4400 50  0001 C CNN
 	1    5100 4400
@@
 F 0 "R8" H 5070 5296 50  0000 L CNN
 F 1 "2k2" H 5070 5205 50  0000 L CNN
-F 2 "" V 4930 5250 50  0001 C CNN
+F 2 "Resistor_THT:R_Axial_DIN0207_L6.3mm_D2.5mm_P2.54mm_Vertical" V 4930 5250 50  0001 C CNN
 F 3 "~" H 5000 5250 50  0001 C CNN
 	1    5000 5250
@@
 F 0 "R11" H 6570 5296 50  0000 L CNN
 F 1 "100R" H 6570 5205 50  0000 L CNN
-F 2 "" V 6430 5250 50  0001 C CNN
+F 2 "Resistor_THT:R_Axial_DIN0207_L6.3mm_D2.5mm_P2.54mm_Vertical" V 6430 5250 50  0001 C CNN
 F 3 "~" H 6500 5250 50  0001 C CNN
 	1    6500 5250
@@
 F 0 "Q8" H 6150 4600 50  0000 L CNN
 F 1 "BC546C" H 6150 4500 50  0000 L CNN
-F 2 "" H 6600 4800 50  0001 C CNN
+F 2 "Package_TO_SOT_THT:TO-92" H 6600 4800 50  0001 C CNN
 F 3 "~" H 6400 4700 50  0001 C CNN
 	1    6400 4700
@@
 F 0 "C2" H 6050 5300 50  0000 L CNN
 F 1 "220pF" H 5900 5200 50  0000 L CNN
-F 2 "" H 6288 5100 50  0001 C CNN
+F 2 "Capacitor_THT:C_Disc_D5.0mm_W2.5mm_P2.50mm" H 6288 5100 50  0001 C CNN
 F 3 "~" H 6250 5250 50  0001 C CNN
 	1    6250 5250
@@
 F 0 "D9" H 6350 4350 50  0000 L CNN
 F 1 "1N914" H 6200 4250 50  0000 L CNN
-F 2 "" H 6250 4400 50  0001 C CNN
+F 2 "Diode_THT:D_DO-35_SOD27_P2.54mm_Vertical_KathodeUp" H 6250 4400 50  0001 C CNN
 F 3 "~" H 6250 4400 50  0001 C CNN
 	1    6250 4400
@@
 F 0 "R5" H 4070 4896 50  0000 L CNN
 F 1 "470R" H 4070 4805 50  0000 L CNN
-F 2 "" V 3930 4850 50  0001 C CNN
+F 2 "Resistor_THT:R_Axial_DIN0207_L6.3mm_D2.5mm_P2.54mm_Vertical" V 3930 4850 50  0001 C CNN
 F 3 "~" H 4000 4850 50  0001 C CNN
 	1    4000 4850
@@
 F 0 "R4" H 3070 4896 50  0000 L CNN
 F 1 "470R" H 3070 4805 50  0000 L CNN
-F 2 "" V 2930 4850 50  0001 C CNN
+F 2 "Resistor_THT:R_Axial_DIN0207_L6.3mm_D2.5mm_P2.54mm_Vertical" V 2930 4850 50  0001 C CNN
 F 3 "~" H 3000 4850 50  0001 C CNN
 	1    3000 4850
@@
 F 0 "RV5" H 3930 5296 50  0000 R CNN
 F 1 "2k" H 3930 5205 50  0000 R CNN
-F 2 "" H 4000 5250 50  0001 C CNN
+F 2 "Potentiometer_THT:Potentiometer_Bourns_3266Z_Horizontal" H 4000 5250 50  0001 C CNN
 F 3 "~" H 4000 5250 50  0001 C CNN
 	1    4000 5250
@@
 F 0 "D7" V 6950 3100 50  0000 L CNN
 F 1 "1N914" V 7050 3100 50  0000 L CNN
-F 2 "" H 7000 3000 50  0001 C CNN
+F 2 "Diode_THT:D_DO-35_SOD27_P2.54mm_Vertical_KathodeUp" H 7000 3000 50  0001 C CNN
 F 3 "~" H 7000 3000 50  0001 C CNN
 	1    7000 3000

Commit message: crude placement
Parts:
- added J1: Imput-, Connector_Pin:Pin_D1.1mm_L8.5mm_W2.5mm_FlatFork, symbol Connector:Conn_01x01_Male
- added J2: Input+, Connector_Pin:Pin_D1.1mm_L8.5mm_W2.5mm_FlatFork, symbol Connector:Conn_01x01_Male
- added J3: V+, Connector_Pin:Pin_D1.1mm_L8.5mm_W2.5mm_FlatFork, symbol Connector:Conn_01x01_Male
- added J4: Output, Connector_Pin:Pin_D1.1mm_L8.5mm_W2.5mm_FlatFork, symbol Connector:Conn_01x01_Male
- added J5: V-, Connector_Pin:Pin_D1.1mm_L8.5mm_W2.5mm_FlatFork, symbol Connector:Conn_01x01_Male
- added J6: GND, Connector_Pin:Pin_D1.1mm_L8.5mm_W2.5mm_FlatFork, symbol Connector:Conn_01x01_Male
- Q10, Q9: footprint Package_TO_SOT_THT:TO-220-3_Vertical -> TAC:to225_std
Connections:
- net labels added: GND
- net labels removed: Input+, Input-, Output, V+, V-
- wire segments 113 -> 115
Other:
- note removed: "O NC"
- moved on the sheet: D1, D2, L1, Q2, Q3

Commit message: abandoned layout. just TAC schematics for DOA socket
Parts:
- removed RV1, RV4, RV5: 2k, Potentiometer_THT:Potentiometer_Bourns_3266Z_Horizontal, symbol Device:R_POT
- R1, R4, R5: value 470R -> 2k2
Connections:
- wire segments 115 -> 103
Changed lines of the file:
@@
 Wire Wire Line
 	7500 5800 7600 5800
-Wire Wire Line
-	4000 5000 4000 5100
-Wire Wire Line
-	4000 5400 4000 5500
-Wire Wire Line
-	3000 5000 3000 5100
-Wire Wire Line
-	3000 5400 3000 5500
-Wire Wire Line
-	3000 5500 3250 5500
-Connection ~ 3250 5500
-Wire Wire Line
-	3250 5250 3250 5500
-Wire Wire Line
-	3150 5250 3250 5250
-Wire Wire Line
-	3750 5500 4000 5500
-Wire Wire Line
-	3250 5500 3750 5500
-Connection ~ 3750 5500
-Wire Wire Line
-	3750 5250 3750 5500
-Wire Wire Line
-	3850 5250 3750 5250
-$Comp
-L Device:R_POT RV5
-U 1 1 5FEB1771
-P 4000 5250
-F 0 "RV5" H 3930 5296 50  0000 R CNN
-F 1 "2k" H 3930 5205 50  0000 R CNN
-F 2 "Potentiometer_THT:Potentiometer_Bourns_3266Z_Horizontal" H 4000 5250 50  0001 C CNN
-F 3 "~" H 4000 5250 50  0001 C CNN
-	1    4000 5250
-	-1   0    0    -1
-$EndComp
-$Comp
-L Device:R_POT RV4
-U 1 1 5FE75F1A
-P 3000 5250
-F 0 "RV4" H 2930 5296 50  0000 R CNN
-F 1 "2k" H 2930 5205 50  0000 R CNN
-F 2 "Potentiometer_THT:Potentiometer_Bourns_3266Z_Horizontal" H 3000 5250 50  0001 C CNN
-F 3 "~" H 3000 5250 50  0001 C CNN
-	1    3000 5250
-	1    0    0    -1
-$EndComp
 $Comp
 L Device:R R5
@@
 P 4000 4850
 F 0 "R5" H 4070 4896 50  0000 L CNN
-F 1 "470R" H 4070 4805 50  0000 L CNN
+F 1 "2k2" H 4070 4805 50  0000 L CNN
 F 2 "Resistor_THT:R_Axial_DIN0207_L6.3mm_D2.5mm_P2.54mm_Vertical" V 3930 4850 50  0001 C CNN
 F 3 "~" H 4000 4850 50  0001 C CNN
@@
 P 3000 4850
 F 0 "R4" H 3070 4896 50  0000 L CNN
-F 1 "470R" H 3070 4805 50  0000 L CNN
+F 1 "2k2" H 3070 4805 50  0000 L CNN
 F 2 "Resistor_THT:R_Axial_DIN0207_L6.3mm_D2.5mm_P2.54mm_Vertical" V 2930 4850 50  0001 C CNN
 F 3 "~" H 3000 4850 50  0001 C CNN
 	1    3000 4850
 	1    0    0    -1
-$EndComp
-Wire Wire Line
-	3500 2000 3500 1900
-Wire Wire Line
-	3500 1600 3500 1500
-Wire Wire Line
-	3750 1500 3850 1500
-Wire Wire Line
-	3500 1500 3750 1500
-Connection ~ 3750 1500
-Wire Wire Line
-	3750 1750 3750 1500
-Wire Wire Line
-	3650 1750 3750 1750
-$Comp
-L Device:R_POT RV1
-U 1 1 5FE73318
-P 3500 1750
-F 0 "RV1" H 3430 1704 50  0000 R CNN
-F 1 "2k" H 3430 1795 50  0000 R CNN
-F 2 "Potentiometer_THT:Potentiometer_Bourns_3266Z_Horizontal" H 3500 1750 50  0001 C CNN
-F 3 "~" H 3500 1750 50  0001 C CNN
-	1    3500 1750
-	1    0    0    1
 $EndComp
 $Comp
@@
 P 4000 1500
 F 0 "R1" V 3793 1500 50  0000 C CNN
-F 1 "470R" V 3884 1500 50  0000 C CNN
+F 1 "2k2" V 3884 1500 50  0000 C CNN
 F 2 "Resistor_THT:R_Axial_DIN0207_L6.3mm_D2.5mm_P2.54mm_Vertical" V 3930 1500 50  0001 C CNN
 F 3 "~" H 4000 1500 50  0001 C CNN
@@
 	0    1    1    0
 $EndComp
+Wire Wire Line
+	3500 1500 3850 1500
+Wire Wire Line
+	3500 1500 3500 2000
+Wire Wire Line
+	3000 5500 4000 5500
+Wire Wire Line
+	3000 5000 3000 5500
+Wire Wire Line
+	4000 5000 4000 5500
 $EndSCHEMATC
