File: TAC_RI279/RI279C.kicad_pcb (KiCad board)
At the start: 2 copper layers, 49 x 39 mm, 10 parts, among them J1 Ribbon Cable, J2 Multiway, J3 Meter

Commit message: status before using KiCad 6.0
Connections:
- SK2 pad RN: Net-(SK2-PadRN) -> unconnected-(SK2-PadRN)
- SK2 pad TN: Net-(SK2-PadTN) -> unconnected-(SK2-PadTN)
- SK3 pad TN: Net-(SK3-PadTN) -> unconnected-(SK3-PadTN)
Other:
- net class Default removed
