File: TAC_GL270D/GL270-DOA2520.kicad_pro/GL270-DOA2520.kicad_pro.kicad_sch (KiCad schematic)
At the start: 227 parts, among them J2 Ribbon Cable, J3 (10k), Q1 2N3904, Q2 2N3904, Q3 2N3906, SW1 +48V On, SW10 SW_QPDT_x4, SW11 SW_QPDT_x4, SW12 SW_QPDT_x4, SW13 SW_QPDT_x4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

Commit message: first iteration DOA Mod circuit diagram
Parts:
- removed #C10, #C11: 22p, symbol Device:C
- removed #C12, #C4: 3300u, symbol GL270-MicIn-rescue:CP-Device
- removed #C13, #C9: 100n, symbol Device:C
- removed #C14, #C5, #C6, #C7, #C8: 47u, symbol GL270-MicIn-rescue:CP-Device
- removed #C15, #C16: 100p, symbol Device:C
- removed #C19: 10p, symbol Device:C
- removed #C20: 10V 100u, symbol GL270-MicIn-rescue:CP-Device
- removed #Q1, #Q2, #Q3, #Q4, #Q5, #Q6: BC560, Package_TO_SOT_THT:TO-92_Inline, symbol Transistor_BJT:BC560
- removed #R1: 1k5, symbol Device:R
- removed #R10, #R8: 6k8, symbol Device:R
- removed #R11, #R7: 3k3, symbol Device:R
- removed #R12, #R13, #R16: 1M, symbol Device:R
- removed #R14: 270R, symbol Device:R
- removed #R18, #R22, #R6: 2k2, symbol Device:R
- removed #R19, #R20: 3k6, symbol Device:R
- removed #R2: 10k, symbol Device:R
- removed #R21: 5R6, symbol Device:R
- removed #R23: 100k, symbol Device:R
- removed #U1: TL072, symbol Amplifier_Operational:TL072
- removed #U2: NE5534, symbol Amplifier_Operational:NE5534
- removed D1, D2, D3, D4, D5, D6: 1N4148, symbol Device:D
- added #C3: 50V 10p, symbol Device:C
- added #CMRR: 2k, symbol GL270-MicIn-rescue:R_POT-Device
- added #RF: 9k1, symbol Device:R
- added #U3: DOA2520, symbol TAC-DOA:DOA2520
- #R1, #R2: value 5R6 -> 10R
- #R4: value 82k -> 10k
- #R5: value 2k2 -> 10R
Connections:
- net #J1: now also #R3.2
- net #J2: now also #R4.2
- net #J3: now also SW7.2 (B), #C3.1, #CMRR.1, #CMRR.2, #U3.3; no longer R15.2, R15.3
- net #J9: now also R15.2, R15.3; no longer SW7.2 (B)
- net GND: now also #R5.2, #U3.5 (0V); no longer #R3.2
- net V+: now also #U3.6 (V+)
- net V-: now also #CMRR.3, #RF.1, #U3.4 (V-); no longer #R4.1
- net at #R3.1: now also #R5.1, #C3.2, #RF.2, #U3.2 (-)
- new net: #R4.1, #U3.1 (+)
- no-connect marks 29 -> 28
Other:
- note added: "Components prefixed # are part of the DOA daughter board."
- note added: "Components prefixed ** are part of the RI277 connector card."
- note added: "DOA 2520 DAUGHTER BOARD"
- note added: "DOA Input Modification PCB: ELI-Diff (Rev 4) by Eli Audio"
- note removed: "Components prefixed # or D are part of the AML daughter board."
- note removed: "Components prefixed ** are part the RI277 connector card."
- note removed: "MIC PREAMP"
- note removed: "Microphone Input Modification PCB: AML-07-048 (Rev 4) by AML & Langley Design"
- company: Riven Hexagon -> Riven Hexagon Electronics
- moved on the sheet: **J0, **J1, **J2, **R2, **R3, *R100, *R105, *R106, *R107, *R108, *R42, *R43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
